Commit message: Balance a triple cart pole using lqr

File: triple_cartpole.urdf (robot description, URDF)
Before this commit: robot DoubleCartPole, 3 links, 3 joints
Links:
- added link pendulum2, mass 2; visual cylinder length=1 radius=.01; visual sphere radius=.05
Joints:
- added joint theta2: type continuous, parent pendulum1, child pendulum2, origin xyz=0 0 1, axis 0 -1 0

Commit message: Alter urdf to make it right

File: triple_cartpole.urdf (robot description, URDF)
Before this commit: robot DoubleCartPole, 4 links, 4 joints
Links:
- link pendulum2: mass 2 -> 1
Joints:
- joint theta2: origin xyz=0 0 1 -> xyz=0 0 -1
